File: effectiveRangeRelay.kicad_sch (KiCad schematic)
At the start: 17 parts, among them J1 RELAY_CTRL, J2 OUT, J3 RELAY_PWR, K1 J107F1CS125VDC.36, Q1 2N7002, U1 APC-817C1-SL

Commit message: fix: removed extra capacitor, fixed url, silk
Parts:
- removed C2: 1uF, Capacitor_SMD:C_0603_1608Metric_Pad1.08x0.95mm_HandSolder, symbol Device:C
- renumbered R6 to R4
Changed lines of the file:
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@@
-	)
-	(junction
-		(at 97.79 120.65)
-		(diameter 0)
-		(color 0 0 0 0)
 	)
 	(junction
@@
 	)
 	(junction
-		(at 97.79 97.79)
-		(diameter 0)
-		(color 0 0 0 0)
-	)
-	(junction
 		(at 220.98 77.47)
 		(diameter 0)
@@
 	(wire
 		(pts
-			(xy 97.79 97.79) (xy 110.49 97.79)
-		)
-		(stroke
-			(width 0)
-			(type default)
-		)
-	)
-	(wire
-		(pts
 			(xy 147.32 121.92) (xy 175.26 121.92)
 		)
@@
 	(wire
 		(pts
-			(xy 97.79 113.03) (xy 97.79 120.65)
-		)
-		(stroke
-			(width 0)
-			(type default)
-		)
-	)
-	(wire
-		(pts
 			(xy 157.48 102.87) (xy 167.64 102.87)
 		)
@@
 	(wire
 		(pts
-			(xy 88.9 120.65) (xy 97.79 120.65)
+			(xy 88.9 120.65) (xy 109.22 120.65)
 		)
 		(stroke
@@
 	(wire
 		(pts
-			(xy 97.79 120.65) (xy 109.22 120.65)
-		)
-		(stroke
-			(width 0)
-			(type default)
-		)
-	)
-	(wire
-		(pts
-			(xy 88.9 97.79) (xy 97.79 97.79)
+			(xy 88.9 97.79) (xy 110.49 97.79)
 		)
 		(stroke
@@
 		(pts
 			(xy 76.2 86.36) (xy 63.5 86.36)
-		)
-		(stroke
-			(width 0)
-			(type default)
-		)
-	)
-	(wire
-		(pts
-			(xy 97.79 97.79) (xy 97.79 105.41)
 		)
 		(stroke
@@
 		(on_board yes)
 		(dnp no)
-		(property "Reference" "R6"
+		(property "Reference" "R4"
 			(at 83.185 106.68 90)
 			(effects
@@
 			(project "effectiveRangeRelay"
 				(path "/6eab7a25-9b20-4eb7-9336-dd2042abdd78"
-					(reference "R6")
+					(reference "R4")
 					(unit 1)
 				)
@@
 					(unit 1)
 				)
-			)
-		)
-	)
-	(symbol
-		(lib_id "Device:C")
-		(at 97.79 109.22 0)
-		(mirror y)
-		(unit 1)
-		(exclude_from_sim no)
-		(in_bom yes)
-		(on_board yes)
-		(dnp no)
-		(property "Reference" "C2"
-			(at 94.615 107.95 0)
-			(effects
-				(font
-					(size 1.27 1.27)
-				)
-				(justify left)
-			)
-		)
-		(property "Value" "1uF"
-			(at 94.615 110.49 0)
-			(effects
-				(font
-					(size 1.27 1.27)
-				)
-				(justify left)
-			)
-		)
-		(property "Footprint" "Capacitor_SMD:C_0603_1608Metric_Pad1.08x0.95mm_HandSolder"
-			(at 96.8248 113.03 0)
-			(effects
-				(font
-					(size 1.27 1.27)
-				)
-				(hide yes)
-			)
-		)
-		(property "Datasheet" "~"
-			(at 97.79 109.22 0)
-			(effects
-				(font
-					(size 1.27 1.27)
-				)
-				(hide yes)
-			)
-		)
-		(property "Description" "Unpolarized capacitor"
-			(at 97.79 109.22 0)
-			(effects
-				(font
-					(size 1.27 1.27)
-				)
-				(hide yes)
-			)
-		)
-		(property "MPN" "GRM188R61A105KA61D"
-			(at 97.79 109.22 0)
-			(effects
-				(font
-					(size 1.27 1.27)
-				)
-				(hide yes)
-			)
-		)
-		(property "Manufaturer" ""
-			(at 97.79 109.22 0)
-			(effects
-				(font
-					(size 1.27 1.27)
-				)
-				(hide yes)
-			)
-		)
-		(pin "1"
-		)
-		(pin "2"
-		)
-		(instances
-			(project "effectiveRangeRelay"
-				(path "/6eab7a25-9b20-4eb7-9336-dd2042abdd78"
-					(reference "C2")
-					(unit 1)
-				)

Commit message: finished initial release
Parts:
- removed D1: TS4148 RCG, Diode_SMD:D_0603_1608Metric, symbol Diode:1N4001
- removed J1: RELAY_CTRL, Connector_PinHeader_2.54mm:PinHeader_1x02_P2.54mm_Vertical, symbol Connector:Conn_01x02_Pin
- removed J2: OUT, relay:CONN_1935174_PXC, symbol Connector:Conn_01x03_Pin
- removed J3: RELAY_PWR, Connector_PinHeader_2.54mm:PinHeader_1x02_P2.54mm_Vertical, symbol Connector:Conn_01x02_Pin
- removed Q1: 2N7002, Package_TO_SOT_SMD:SOT-23, symbol Transistor_FET:2N7002
- removed R1, R5: 180, Resistor_SMD:R_0603_1608Metric, symbol Device:R
- removed R4: 1M, Resistor_SMD:R_0603_1608Metric, symbol Device:R
- removed U1: APC-817C1-SL, relay:APC-817C1-SL, symbol Isolator:NSL-32
- added D101, D102: D_Schottky, Diode_SMD:D_SOD-882, symbol Device:D_Schottky
- added J101: Screw_Terminal_01x02, TerminalBlock_CUI:TerminalBlock_CUI_TB007-508-02_1x02_P5.08mm_Horizontal, symbol Connector:Screw_Terminal_01x02
- added J102: Conn_01x02, relay:CONN02_533750210_MOL, symbol Connector_Generic:Conn_01x02
- added J103, J104: Screw_Terminal_01x05, TerminalBlock_CUI:TerminalBlock_CUI_TB007-508-05_1x05_P5.08mm_Horizontal, symbol Connector:Screw_Terminal_01x05
- added J105: Conn_01x22_Female, relay:Hirose_FH12-22S-0.5SH_1x22-1MP_P0.50mm_Horizontal, symbol Connector:Conn_01x22_Socket
- added K102: J107F1CS125VDC.36, relay:RELAY5_J107F-1C_CRS, symbol relay:J107F1CS125VDC.36
- added NT101, NT102: NetTie_2, NetTie:NetTie-2_SMD_Pad2.0mm, symbol Device:NetTie_2
- added R103: 1k, Resistor_SMD:R_0402_1005Metric, symbol Device:R
- added R104: 1M, Resistor_SMD:R_0402_1005Metric, symbol Device:R
- added U101: GSF7002DW, relay:GSF7002DW, symbol relay:GSF7002DW
- R101: renamed from R3; footprint Resistor_SMD:R_0603_1608Metric -> Resistor_SMD:R_0402_1005Metric
- R102: renamed from R2; value 180 -> 1k; footprint Resistor_SMD:R_0603_1608Metric -> Resistor_SMD:R_0402_1005Metric
- renumbered H1 to H101, H3 to H102, H2 to H103, H4 to H104, K1 to K101
Connections:
- net GND2 is gone; now on net GND: R101.2
- net +5V: now also D101.1 (K), D102.1 (K), J105.2 (Pin_2), K102.5
- net GND: now also J105.1 (Pin_1), J105.10 (Pin_10), J105.13 (Pin_13), J105.16 (Pin_16), J105.19 (Pin_19), J105.4 (Pin_4), J105.7 (Pin_7), R104.2, U101.S1, U101.S2
- net COIL_CTRL renamed COIL1_CTRL
- net COIL1_CTRL: now also J105.3 (Pin_3)
- net COM renamed COM1
- net COM1: now also J103.3 (Pin_3)
- net NC renamed NC1
- net NC1: now also J103.4 (Pin_4)
- net NO renamed NO1
- net NO1: now also J103.2 (Pin_2)
- net Q_BASE: no longer names the net of R102.1
- net Q_BASE: now also U101.G1
- net Q_COLL renamed Q_COLL1
- net Q_COLL1: now also D101.2 (A), U101.D1
- new net: R103.1, U101.G2
- new net COIL2_CTRL: J105.5 (Pin_5), R103.2, R104.1
- new net COM2: J104.3 (Pin_3), K102.1
- new net EXT_3V: J105.22 (Pin_22)
- new net EXT_INT: J105.6 (Pin_6)
- new net GND1: J101.2 (Pin_2), J103.5 (Pin_5), J104.5 (Pin_5), NT101.1
- new net GND_TAP: J102.1 (Pin_1), NT101.2
- new net ICSP_EXT.CLK: J105.9 (Pin_9)
- new net ICSP_EXT.DAT: J105.8 (Pin_8)
- new net ICSP_EXT.VDD: J105.12 (Pin_12)
- new net ICSP_EXT.~{MCLR}: J105.11 (Pin_11)
- new net NC2: J104.4 (Pin_4), K102.4
- new net NO2: J104.2 (Pin_2), K102.3
- new net Q_COLL2: D102.2 (A), K102.2, U101.D2
- new net SCL_EXT: J105.20 (Pin_20)
- new net SDA_EXT: J105.21 (Pin_21)
- new net SPI_EXT.MISO: J105.15 (Pin_15)
- new net SPI_EXT.MOSI: J105.17 (Pin_17)
- new net SPI_EXT.SCLK: J105.18 (Pin_18)
- new net SPI_EXT.~{CE}: J105.14 (Pin_14)
- new net VAA: J101.1 (Pin_1), J103.1 (Pin_1), J104.1 (Pin_1), NT102.1
- new net VAA_TAP: J102.2 (Pin_2), NT102.2
- no-connect marks 0 -> 12
Other:
- moved on the sheet: K101, R101, R102

Commit message: fix legend
Other:
- title: Effective Range RelayDevice -> Effective Range RelayDeviceDual
Changed lines of the file:
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@@
 	(paper "A4")
 	(title_block
-		(title "Effective Range RelayDevice")
+		(title "Effective Range RelayDeviceDual")
 		(date "2026-03-19")
-		(rev "v2.1.0")
+		(rev "v0.1.0")
 		(company "Effective Range Kft")
 		(comment 1 "visit https://creativecommons.org/licenses/by/4.0/")
 		(comment 2 "is licensed under CC BY 4.0. To view a copy of this license,")
-		(comment 3 "License: MrHAT © 2024 by Ferenc Nandor Janky & Attila Gombos")
+		(comment 3 "License: MrHAT © 2024 by Ferenc Nandor Janky & Attila Gombos & Tamas Janky")
 		(comment 4 "Design Engineer: Ferenc Janky")
 	)

Commit message: rework
Connections:
- net NC1: now also J103.2 (Pin_2); no longer J103.4 (Pin_4)
- net NO1: now also J103.4 (Pin_4); no longer J103.2 (Pin_2)
Changed lines of the file:
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@@
 	)
 	(label "NO1"
-		(at 240.03 104.14 180)
+		(at 240.03 109.22 180)
 		(effects
 			(font
@@
 	)
 	(label "NC1"
-		(at 240.03 109.22 180)
+		(at 240.03 104.14 180)
 		(effects
 			(font
